Commit message: [WIP] Test inertia

File: urdf/robot.xacro (robot description, xacro)
@@ -10,8 +10,20 @@
   <color rgba="0 1 0 1" />
 </material>
+<xacro:property name="inertiaTest" value="0.1" />
 <xacro:property name="bodyLen" value="0.6" />
 <xacro:property name="bodyWidth" value="0.3" />
 <xacro:property name="bodyHeight" value="0.15" />
+<link name="world"/>
+<joint name="fixed" type="fixed">
+    <origin xyz="0 0 2" rpy="0 0 0"/>
+    <parent link="world"/>
+    <child link="base_link"/>
+</joint>
 <link name="base_link">
+  <inertial>
+    <origin xyz="0 0 0" rpy="0 0 0"/>
+    <mass value="1"/>
+    <inertia ixx="${inertiaTest}" ixy="0" ixz="0" iyy="${inertiaTest}" iyz = "0" izz="${inertiaTest}" />
+  </inertial>
   <visual>
     <origin xyz="0 0 0" rpy="0 0 0" />
@@ -23,7 +35,18 @@
     </material>
   </visual>
+  <collision>
+    <origin xyz="0 0 0" rpy="0 0 0" />
+    <geometry>
+      <box size="${bodyLen} ${bodyWidth} ${bodyHeight}"/>
+    </geometry>
+  </collision>
 </link>
 <xacro:macro name="leg" params="prefix side front">
   <link name="shoulder_${prefix}_link">
+    <inertial>
+      <origin xyz="0 0 0" rpy="0 0 0"/>
+      <mass value="0.1"/>
+      <inertia ixx="${inertiaTest}" ixy="0" ixz="0" iyy="${inertiaTest}" iyz = "0" izz="${inertiaTest}" />
+    </inertial>
     <visual>
       <origin xyz="0 ${side*0.05} 0" rpy="0 0 0" />
@@ -33,4 +56,10 @@
       <material name="red"/>
     </visual>
+    <collision>
+      <origin xyz="0 ${side*0.05} 0" rpy="0 0 0" />
+      <geometry>
+        <box size="0.1 0.1 0.1" />
+      </geometry>
+    </collision>
   </link>
   <joint name="baseToShoulder_${prefix}_joint" type="revolute">
@@ -39,7 +68,12 @@
     <child link="shoulder_${prefix}_link" />
     <axis xyz="1 0 0" />
-    <limit upper="3.14" lower="-3.14" effort="10" velocity="10"/>
+    <limit upper="${pi/4}" lower="${-pi/4}" effort="10" velocity="10"/>
   </joint>
   <link name="thigh_${prefix}_link">
+    <inertial>
+      <origin xyz="0 0 0" rpy="0 0 0"/>
+      <mass value="0.15"/>
+      <inertia ixx="${inertiaTest}" ixy="0" ixz="0" iyy="${inertiaTest}" iyz = "0" izz="${inertiaTest}" />
+    </inertial>
     <visual>
       <origin xyz="0 ${side*0.05} -0.05" rpy="0 0 0" />
@@ -49,4 +83,10 @@
       <material name="green"/>
     </visual>
+    <collision>
+      <origin xyz="0 ${side*0.05} -0.05" rpy="0 0 0" />
+      <geometry>
+        <box size="0.1 0.1 0.2" />
+      </geometry>
+    </collision>
   </link>
   <joint name="shoulderToThigh_${prefix}_joint" type="revolute">
@@ -58,4 +98,9 @@
   </joint>
   <link name="tibia_${prefix}_link">
+    <inertial>
+      <origin xyz="0 0 0" rpy="0 0 0"/>
+      <mass value="0.15"/>
+      <inertia ixx="${inertiaTest}" ixy="0" ixz="0" iyy="${inertiaTest}" iyz = "0" izz="${inertiaTest}" />
+    </inertial>
     <visual>
       <origin xyz ="0 0 -0.125" rpy="0 0 0" />
@@ -65,4 +110,10 @@
       <material name="blue"/>
     </visual>
+    <collision>
+      <origin xyz ="0 0 -0.125" rpy="0 0 0" />
+      <geometry>
+        <box size="0.1 0.1 0.25" />
+      </geometry>
+    </collision>
   </link>
   <joint name="tighToTibia_${prefix}_joint" type="revolute">
