Commit message: Starting point of ros2_control_implementation

File: urdf/robot.urdf (robot description, URDF)
Before this commit: robot Unknown Bot, 13 links, 12 joints
Links:
- added link world
- link base_link: mass None -> 1; geometry collision box size=0.6 0.3 0.15; visual box size=0.6 0.3 0.15
- link shoulder_bl_link: mass None -> 0.1; geometry collision box size=0.1 0.1 0.1; visual box size=0.1 0.1 0.1
- link shoulder_br_link: mass None -> 0.1; geometry collision box size=0.1 0.1 0.1; visual box size=0.1 0.1 0.1
- link shoulder_fl_link: mass None -> 0.1; geometry collision box size=0.1 0.1 0.1; visual box size=0.1 0.1 0.1
- link shoulder_fr_link: mass None -> 0.1; geometry collision box size=0.1 0.1 0.1; visual box size=0.1 0.1 0.1
- link thigh_bl_link: mass None -> 0.15; geometry collision box size=0.1 0.1 0.2; visual box size=0.1 0.1 0.2
- link thigh_br_link: mass None -> 0.15; geometry collision box size=0.1 0.1 0.2; visual box size=0.1 0.1 0.2
- link thigh_fl_link: mass None -> 0.15; geometry collision box size=0.1 0.1 0.2; visual box size=0.1 0.1 0.2
- link thigh_fr_link: mass None -> 0.15; geometry collision box size=0.1 0.1 0.2; visual box size=0.1 0.1 0.2
- link tibia_bl_link: mass None -> 0.15; geometry collision box size=0.1 0.1 0.25; visual box size=0.1 0.1 0.25
- link tibia_br_link: mass None -> 0.15; geometry collision box size=0.1 0.1 0.25; visual box size=0.1 0.1 0.25
- link tibia_fl_link: mass None -> 0.15; geometry collision box size=0.1 0.1 0.25; visual box size=0.1 0.1 0.25
- link tibia_fr_link: mass None -> 0.15; geometry collision box size=0.1 0.1 0.25; visual box size=0.1 0.1 0.25
Joints:
- added joint fixed: type fixed, parent world, child base_link, origin xyz=0 0 2 rpy=0 0 0
- joint baseToShoulder_bl_joint: limit lower=-3.14 upper=3.14 effort=10 velocity=10 -> lower=-0.7853981633974483 upper=0.7853981633974483 effort=10 velocity=10
- joint baseToShoulder_br_joint: limit lower=-3.14 upper=3.14 effort=10 velocity=10 -> lower=-0.7853981633974483 upper=0.7853981633974483 effort=10 velocity=10
- joint baseToShoulder_fl_joint: limit lower=-3.14 upper=3.14 effort=10 velocity=10 -> lower=-0.7853981633974483 upper=0.7853981633974483 effort=10 velocity=10
- joint baseToShoulder_fr_joint: limit lower=-3.14 upper=3.14 effort=10 velocity=10 -> lower=-0.7853981633974483 upper=0.7853981633974483 effort=10 velocity=10
