Commit message: First version of quadruped + ros2 control + ignition fortress

File: robot_description/urdf/oneDofBot_description.urdf.xacro (robot description, xacro)
@@ -18,4 +18,5 @@
         <xacro:property name="upper_length" value="0.1" />
         <xacro:property name="upper_height" value="0.5" />
+        <xacro:property name="inertiaTest" value="0.1" />
         <joint name="fixed_joint" type="fixed">
             <parent link="world" />
@@ -31,4 +32,9 @@
                 <material name="red" />
             </visual>
+            <inertial>
+                <origin xyz="0 0 0" rpy="0 0 0"/>
+                <mass value="1"/>
+                <inertia ixx="${inertiaTest}" ixy="0" ixz="0" iyy="${inertiaTest}" iyz = "0" izz="${inertiaTest}" />
+            </inertial>
         </link>
         <joint name="dof_joint" type="continuous" >
@@ -36,4 +42,5 @@
             <child link="upper_link" />
             <origin xyz="0 ${base_width/2} ${base_height - 0.1}" />
+            <dynamics damping="0.0" friction="0.0"/>
         </joint>
         <link name="upper_link">
@@ -45,4 +52,9 @@
                 <material name="blue" />
             </visual>
+            <inertial>
+                <origin xyz="0 0 0" rpy="0 0 0"/>
+                <mass value="1"/>
+                <inertia ixx="${inertiaTest}" ixy="0" ixz="0" iyy="${inertiaTest}" iyz = "0" izz="${inertiaTest}" />
+            </inertial>
         </link>
     </xacro:macro>

File: robot_description/urdf/oneDof_ros2_simulated.urdf.xacro (robot description, xacro)
@@ -2,21 +2,16 @@
 <robot xmlns:xacro="http://www.ros.org/wiki/xacro">
     <xacro:macro name="oneDof_ros2_control">
-        <ros2_control name="oneDof_bot" type="system">
+        <ros2_control name="IgnitionSystem" type="system">
             <hardware>
-                <plugin>robot_hardware/OneDofSimplePosition</plugin>
-                <param name="test_param">3</param>
+                <plugin>ign_ros2_control/IgnitionSystem</plugin>
             </hardware>
             <joint name="dof_joint">
-                <command_interface name="position">
-                    <param name="min">-3.14</param>
-                    <param name="max">3.14</param>
-                </command_interface>
+                <command_interface name="position"/>
                 <state_interface name="position" />
+                <state_interface name="velocity" />
             </joint>
         </ros2_control>
         <gazebo>
             <plugin filename="libign_ros2_control-system.so" name="ign_ros2_control::IgnitionROS2ControlPlugin">
-                <robot_param>robot_description</robot_param>
-                <robot_param_node>robot_state_publisher</robot_param_node>
                 <parameters>$(find robot_urdf)/oneDof_simple_controllers.yaml</parameters>
             </plugin>

File: robot_description/urdf/quadruped_description.urdf.xacro (robot description, xacro)
@@ -14,32 +14,34 @@
 <xacro:property name="bodyWidth" value="0.3" />
 <xacro:property name="bodyHeight" value="0.15" />
-<link name="world"/>
-<joint name="fixed" type="fixed">
-    <origin xyz="0 0 2" rpy="0 0 0"/>
-    <parent link="world"/>
-    <child link="base_link"/>
-</joint>
-<link name="base_link">
-  <inertial>
-    <origin xyz="0 0 0" rpy="0 0 0"/>
-    <mass value="1"/>
-    <inertia ixx="${inertiaTest}" ixy="0" ixz="0" iyy="${inertiaTest}" iyz = "0" izz="${inertiaTest}" />
-  </inertial>
-  <visual>
-    <origin xyz="0 0 0" rpy="0 0 0" />
-    <geometry>
-      <box size="${bodyLen} ${bodyWidth} ${bodyHeight}"/>
-    </geometry>
-    <material name="white">
-      <color rgba="1 1 1 1" />
-    </material>
-  </visual>
-  <collision>
-    <origin xyz="0 0 0" rpy="0 0 0" />
-    <geometry>
-      <box size="${bodyLen} ${bodyWidth} ${bodyHeight}"/>
-    </geometry>
-  </collision>
-</link>
+<xacro:macro name="body">
+    <link name="world"/>
+    <joint name="fixed" type="fixed">
+        <origin xyz="0 0 2" rpy="0 0 0"/>
+        <parent link="world"/>
+        <child link="base_link"/>
+    </joint>
+    <link name="base_link">
+      <inertial>
+        <origin xyz="0 0 0" rpy="0 0 0"/>
+        <mass value="1"/>
+        <inertia ixx="${inertiaTest}" ixy="0" ixz="0" iyy="${inertiaTest}" iyz = "0" izz="${inertiaTest}" />
+      </inertial>
+      <visual>
+        <origin xyz="0 0 0" rpy="0 0 0" />
+        <geometry>
+          <box size="${bodyLen} ${bodyWidth} ${bodyHeight}"/>
+        </geometry>
+        <material name="white">
+          <color rgba="1 1 1 1" />
+        </material>
+      </visual>
+      <collision>
+        <origin xyz="0 0 0" rpy="0 0 0" />
+        <geometry>
+          <box size="${bodyLen} ${bodyWidth} ${bodyHeight}"/>
+        </geometry>
+      </collision>
+  </link>
+</xacro:macro>
 <xacro:macro name="leg" params="prefix side front">
   <link name="shoulder_${prefix}_link">
@@ -117,15 +119,11 @@
     </collision>
   </link>
-  <joint name="tighToTibia_${prefix}_joint" type="revolute">
+  <joint name="thighToTibia_${prefix}_joint" type="revolute">
     <origin xyz ="0 ${side*0.05} -0.15" rpy="0 -0.77 0" />
     <parent link="thigh_${prefix}_link" />
     <child link="tibia_${prefix}_link" />
-    <axis xyz="0 1 0" />:
+    <axis xyz="0 1 0" />
     <limit upper="3.14" lower="-3.14" effort="10" velocity="10"/>
   </joint>
 </xacro:macro>
-<xacro:leg prefix="bl" side="1" front="-1"/>
-<xacro:leg prefix="br" side="-1" front="-1"/>
-<xacro:leg prefix="fl" side="1" front="1"/>
-<xacro:leg prefix="fr" side="-1" front="1"/>
 </robot>

File: robot_description/urdf/test.urdf.xacro (robot description, xacro)
@@ -1,7 +1,9 @@
 <?xml version="0.1"?>
 <robot xmlns:xacro="http://www.ros.org/wiki/xacro" name="1 DoF Bot">
-    <!-- <xacro:include filename="$(find robot_urdf)/urdf/oneDofBot_description.urdf.xacro" /> -->
-    <xacro:include filename="oneDofBot_description.urdf.xacro" />
+    <xacro:include filename="$(find robot_urdf)/oneDofBot_description.urdf.xacro" />
+    <xacro:include filename="$(find robot_urdf)/oneDof_ros2_control.urdf.xacro" />
+    <!-- <xacro:include filename="oneDofBot_description.urdf.xacro" />
     <xacro:include filename="oneDof_ros2_control.urdf.xacro" />
+    -->
     <xacro:bot_description />
     <xacro:oneDof_ros2_control/>
